File: blankproject.kicad_pcb (KiCad board)
At the start: 2 copper layers, 160 x 100 mm, 4 parts

Commit message: Started assembling librarys
Parts:
- removed MH1, MH2, MH3, MH4: MountingHole_2.7mm_M2.5_DIN965, MountingHole:MountingHole_2.7mm_M2.5_DIN965
Other:
- board outline removed
- board text removed: "Mounting holes are optional Keepout areas are for for guide rails"
Changed lines of the file:
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@@
   )
   (paper "A4")
+  (title_block
+    (date "2022-11-16")
+    (company "SquashedFly")
+  )
   (layers
     (0 "F.Cu" signal)
@@
     (48 "B.Fab" user)
     (49 "F.Fab" user)
+    (50 "User.1" user)
+    (51 "User.2" user)
+    (52 "User.3" user)
+    (53 "User.4" user)
+    (54 "User.5" user)
+    (55 "User.6" user)
+    (56 "User.7" user)
+    (57 "User.8" user)
+    (58 "User.9" user)
   )
   (setup
-    (stackup
-      (layer "F.SilkS" (type "Top Silk Screen"))
-      (layer "F.Paste" (type "Top Solder Paste"))
-      (layer "F.Mask" (type "Top Solder Mask") (color "Green") (thickness 0.01))
-      (layer "F.Cu" (type "copper") (thickness 0.035))
-      (layer "dielectric 1" (type "core") (thickness 1.51) (material "FR4") (epsilon_r 4.5) (loss_tangent 0.02))
-      (layer "B.Cu" (type "copper") (thickness 0.035))
-      (layer "B.Mask" (type "Bottom Solder Mask") (color "Green") (thickness 0.01))
-      (layer "B.Paste" (type "Bottom Solder Paste"))
-      (layer "B.SilkS" (type "Bottom Silk Screen"))
-      (copper_finish "None")
-      (dielectric_constraints no)
-    )
     (pad_to_mask_clearance 0)
-    (aux_axis_origin 55 145)
-    (grid_origin 55 145)
     (pcbplotparams
-      (layerselection 0x0000030_ffffffff)
+      (layerselection 0x00010fc_ffffffff)
       (disableapertmacros false)
       (usegerberextensions false)
@@
       (outputformat 1)
       (mirror false)
-      (drillshape 0)
+      (drillshape 1)
       (scaleselection 1)
       (outputdirectory "")
@@
   )
   (net 0 "")
-  (footprint "MountingHole:MountingHole_2.7mm_M2.5_DIN965" locked (layer "F.Cu")
-    (at 212.24 139.45)
-    (descr "Mounting Hole 2.7mm, no annular, M2.5, DIN965")
-    (tags "mounting hole 2.7mm no annular m2.5 din965")
-    (attr exclude_from_pos_files exclude_from_bom)
-    (fp_text reference "MH4" (at 0 -3.35) (layer "F.SilkS") hide
-      (effects (font (size 1 1) (thickness 0.15)))
-    )
-    (fp_text value "MountingHole_2.7mm_M2.5_DIN965" (at 0 3.35) (layer "F.Fab") hide
-      (effects (font (size 1 1) (thickness 0.15)))
-    )
-    (fp_text user "${REFERENCE}" (at 0.3 0) (layer "F.Fab") hide
-      (effects (font (size 1 1) (thickness 0.15)))
-    )
-    (fp_circle (center 0 0) (end 2.35 0) (layer "Cmts.User") (width 0.15) (fill none))
-    (fp_circle (center 0 0) (end 2.6 0) (layer "F.CrtYd") (width 0.05) (fill none))
-    (pad "" np_thru_hole circle locked (at 0 0) (size 2.7 2.7) (drill 2.7) (layers *.Cu *.Mask))
-  )
-  (footprint "MountingHole:MountingHole_2.7mm_M2.5_DIN965" (layer "F.Cu")
-    (at 58.57 50.55)
-    (descr "Mounting Hole 2.7mm, no annular, M2.5, DIN965")
-    (tags "mounting hole 2.7mm no annular m2.5 din965")
-    (attr exclude_from_pos_files exclude_from_bom)
-    (fp_text reference "MH1" (at 0 -3.35) (layer "F.SilkS") hide
-      (effects (font (size 1 1) (thickness 0.15)))
-    )
-    (fp_text value "MountingHole_2.7mm_M2.5_DIN965" (at 0 3.35) (layer "F.Fab") hide
-      (effects (font (size 1 1) (thickness 0.15)))
-    )
-    (fp_text user "${REFERENCE}" (at 0.3 0) (layer "F.Fab") hide
-      (effects (font (size 1 1) (thickness 0.15)))
-    )
-    (fp_circle (center 0 0) (end 2.35 0) (layer "Cmts.User") (width 0.15) (fill none))
-    (fp_circle (center 0 0) (end 2.6 0) (layer "F.CrtYd") (width 0.05) (fill none))
-    (pad "" np_thru_hole circle locked (at 0 0) (size 2.7 2.7) (drill 2.7) (layers *.Cu *.Mask))
-  )
-  (footprint "MountingHole:MountingHole_2.7mm_M2.5_DIN965" locked (layer "F.Cu")
-    (at 58.57 139.45)
-    (descr "Mounting Hole 2.7mm, no annular, M2.5, DIN965")
-    (tags "mounting hole 2.7mm no annular m2.5 din965")
-    (attr exclude_from_pos_files exclude_from_bom)
-    (fp_text reference "MH2" (at 0 -3.35) (layer "F.SilkS") hide
-      (effects (font (size 1 1) (thickness 0.15)))
-    )
-    (fp_text value "MountingHole_2.7mm_M2.5_DIN965" (at 0 3.35) (layer "F.Fab") hide
-      (effects (font (size 1 1) (thickness 0.15)))
-    )
-    (fp_text user "${REFERENCE}" (at 0.3 0) (layer "F.Fab") hide
-      (effects (font (size 1 1) (thickness 0.15)))
-    )
-    (fp_circle (center 0 0) (end 2.35 0) (layer "Cmts.User") (width 0.15) (fill none))
-    (fp_circle (center 0 0) (end 2.6 0) (layer "F.CrtYd") (width 0.05) (fill none))
-    (pad "" np_thru_hole circle locked (at 0 0) (size 2.7 2.7) (drill 2.7) (layers *.Cu *.Mask))
-  )
-  (footprint "MountingHole:MountingHole_2.7mm_M2.5_DIN965" locked (layer "F.Cu")
-    (at 212.24 50.55)
-    (descr "Mounting Hole 2.7mm, no annular, M2.5, DIN965")
-    (tags "mounting hole 2.7mm no annular m2.5 din965")
-    (attr exclude_from_pos_files exclude_from_bom)
-    (fp_text reference "MH3" (at 0 -3.35) (layer "F.SilkS") hide
-      (effects (font (size 1 1) (thickness 0.15)))
-    )
-    (fp_text value "MountingHole_2.7mm_M2.5_DIN965" (at 0 3.35) (layer "F.Fab") hide
-      (effects (font (size 1 1) (thickness 0.15)))
-    )
-    (fp_text user "${REFERENCE}" (at 0.3 0) (layer "F.Fab") hide
-      (effects (font (size 1 1) (thickness 0.15)))
-    )
-    (fp_circle (center 0 0) (end 2.35 0) (layer "Cmts.User") (width 0.15) (fill none))
-    (fp_circle (center 0 0) (end 2.6 0) (layer "F.CrtYd") (width 0.05) (fill none))
-    (pad "" np_thru_hole circle locked (at 0 0) (size 2.7 2.7) (drill 2.7) (layers *.Cu *.Mask))
-  )
-  (gr_rect locked (start 55 145) (end 215 45) (layer "Edge.Cuts") (width 0.15) (fill none))
-  (gr_text "Mounting holes are optional\nKeepout areas are for for guide rails" (at 55.5 148) (layer "Cmts.User")
-    (effects (font (size 1 1) (thickness 0.15)) (justify left))
-  )
-  (zone (net 0) (net_name "") (layers F&B.Cu) (hatch full 0.508)
-    (connect_pads (clearance 0))
-    (min_thickness 0.254)
-    (keepout (tracks not_allowed) (vias not_allowed) (pads not_allowed ) (copperpour allowed) (footprints not_allowed))
-    (fill (thermal_gap 0.508) (thermal_bridge_width 0.508))
-    (polygon
-      (pts
-        (xy 215 145)
-        (xy 55 145)
-        (xy 55 142.5)
-        (xy 215 142.5)
-      )
-    )
-  )
-  (zone (net 0) (net_name "") (layers F&B.Cu) (hatch full 0.508)
-    (connect_pads (clearance 0))
-    (min_thickness 0.254)
-    (keepout (tracks not_allowed) (vias not_allowed) (pads not_allowed ) (copperpour allowed) (footprints not_allowed))
-    (fill (thermal_gap 0.508) (thermal_bridge_width 0.508))
-    (polygon
-      (pts
-        (xy 215 47.5)
-        (xy 55 47.5)
-        (xy 55 45)
-        (xy 215 45)
-      )
-    )
-  )
 )
