File: blankproject.kicad_pcb (KiCad board)
At the start: 2 copper layers, 0 parts

Commit message: some edits
Other:
- copper layers 2 -> 4
- board text added: "Following IPC 2221 recomendations, if this PCB is to carry high currents the outside copper layers shall be composed of 2 Oz CU. See other notes to the righ hand side of the schematic above."
Changed lines of the file:
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@@
 (kicad_pcb (version 20211014) (generator pcbnew)
   (general
-    (thickness 1.6)
+    (thickness 4.69)
   )
   (paper "A4")
@@
   )
   (layers
-    (0 "F.Cu" signal)
-    (31 "B.Cu" signal)
+    (0 "F.Cu" mixed)
+    (1 "In1.Cu" mixed)
+    (2 "In2.Cu" mixed)
+    (31 "B.Cu" power)
     (32 "B.Adhes" user "B.Adhesive")
     (33 "F.Adhes" user "F.Adhesive")
@@
     (38 "B.Mask" user)
     (39 "F.Mask" user)
-    (40 "Dwgs.User" user "User.Drawings")
-    (41 "Cmts.User" user "User.Comments")
-    (42 "Eco1.User" user "User.Eco1")
-    (43 "Eco2.User" user "User.Eco2")
+    (41 "Cmts.User" user "Comments")
     (44 "Edge.Cuts" user)
     (45 "Margin" user)
@@
     (48 "B.Fab" user)
     (49 "F.Fab" user)
-    (50 "User.1" user)
-    (51 "User.2" user)
-    (52 "User.3" user)
-    (53 "User.4" user)
-    (54 "User.5" user)
-    (55 "User.6" user)
-    (56 "User.7" user)
-    (57 "User.8" user)
-    (58 "User.9" user)
   )
   (setup
+    (stackup
+      (layer "F.SilkS" (type "Top Silk Screen"))
+      (layer "F.Paste" (type "Top Solder Paste"))
+      (layer "F.Mask" (type "Top Solder Mask") (thickness 0.01))
+      (layer "F.Cu" (type "copper") (thickness 0.035))
+      (layer "dielectric 1" (type "core") (thickness 1.51) (material "FR4") (epsilon_r 4.5) (loss_tangent 0.02))
+      (layer "In1.Cu" (type "copper") (thickness 0.035))
+      (layer "dielectric 2" (type "prepreg") (thickness 1.51) (material "FR4") (epsilon_r 4.5) (loss_tangent 0.02))
+      (layer "In2.Cu" (type "copper") (thickness 0.035))
+      (layer "dielectric 3" (type "core") (thickness 1.51) (material "FR4") (epsilon_r 4.5) (loss_tangent 0.02))
+      (layer "B.Cu" (type "copper") (thickness 0.035))
+      (layer "B.Mask" (type "Bottom Solder Mask") (thickness 0.01))
+      (layer "B.Paste" (type "Bottom Solder Paste"))
+      (layer "B.SilkS" (type "Bottom Silk Screen"))
+      (copper_finish "None")
+      (dielectric_constraints no)
+    )
     (pad_to_mask_clearance 0)
     (pcbplotparams
@@
   )
   (net 0 "")
+  (gr_text "Following IPC 2221 recomendations, if this PCB is to carry high currents the \noutside copper layers shall be composed of 2 Oz CU.\n\nSee other notes to the righ hand side of the schematic above." (at 185.25 178.75) (layer "Cmts.User")
+    (effects (font (size 1.5 1.5) (thickness 0.3)) (justify left))
+  )
 )

Commit message: added JLC minimum track sizes
Other:
- board text removed: "Following IPC 2221 recomendations, if this PCB is to carry high currents the outside copper layers shall be composed of 2 Oz CU. See other notes to the righ hand side of the schematic above."
Changed lines of the file:
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@@
   )
   (net 0 "")
-  (gr_text "Following IPC 2221 recomendations, if this PCB is to carry high currents the \noutside copper layers shall be composed of 2 Oz CU.\n\nSee other notes to the righ hand side of the schematic above." (at 185.25 178.75) (layer "Cmts.User")
-    (effects (font (size 1.5 1.5) (thickness 0.3)) (justify left))
-  )
 )
