File: blankproject.kicad_sch (KiCad schematic)
At the start: 0 parts

Commit message: Started assembling librarys
Other:
- company: (none) -> SquashedFly
Changed lines of the file:
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@@
 (kicad_sch (version 20211123) (generator eeschema)
   (paper "A4")
+  (title_block
+    (date "2022-11-16")
+    (company "SquashedFly")
+  )
   (sheet_instances
     (path "/" (page "1"))
