File: blankproject.kicad_sch (KiCad schematic)
At the start: 0 parts

Commit message: updates - may need reverted
Parts:
- added J?: Screw_Terminal_01x01, symbol Wire to Board:Screw_Terminal_01x01
Changed lines of the file:
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@@
     (company "SquashedFly")
+  )
+  (symbol (lib_id "Wire to Board:Screw_Terminal_01x01") (at 125.73 92.71 0) (unit 1)
+    (in_bom yes) (on_board yes) (fields_autoplaced)
+    (property "Reference" "J?" (id 0) (at 128.27 91.4399 0)
+      (effects (font (size 1.27 1.27)) (justify left))
+    )
+    (property "Value" "Screw_Terminal_01x01" (id 1) (at 128.27 93.9799 0)
+      (effects (font (size 1.27 1.27)) (justify left))
+    )
+    (property "Footprint" "" (id 2) (at 125.73 92.71 0)
+      (effects (font (size 1.27 1.27)) hide)
+    )
+    (property "Datasheet" "https://labbook.skippy.org.uk/projects/kicad/screw" (id 3) (at 125.73 92.71 0)
+      (effects (font (size 1.27 1.27)) hide)
+    )
+    (pin "1")
   )
   (sheet_instances
     (path "/" (page "1"))
   )
+  (symbol_instances
+    (path "/9fa81b1d-9622-4bc6-8198-4b4bc1b152f4"
+      (reference "J?") (unit 1) (value "Screw_Terminal_01x01") (footprint "")
+    )
+  )
 )

Commit message: cleanup
Parts:
- removed J?: Screw_Terminal_01x01, symbol Wire to Board:Screw_Terminal_01x01
Changed lines of the file:
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@@
     (company "SquashedFly")
-  )
-  (symbol (lib_id "Wire to Board:Screw_Terminal_01x01") (at 125.73 92.71 0) (unit 1)
-    (in_bom yes) (on_board yes) (fields_autoplaced)
-    (property "Reference" "J?" (id 0) (at 128.27 91.4399 0)
-      (effects (font (size 1.27 1.27)) (justify left))
-    )
-    (property "Value" "Screw_Terminal_01x01" (id 1) (at 128.27 93.9799 0)
-      (effects (font (size 1.27 1.27)) (justify left))
-    )
-    (property "Footprint" "" (id 2) (at 125.73 92.71 0)
-      (effects (font (size 1.27 1.27)) hide)
-    )
-    (property "Datasheet" "https://labbook.skippy.org.uk/projects/kicad/screw" (id 3) (at 125.73 92.71 0)
-      (effects (font (size 1.27 1.27)) hide)
-    )
-    (pin "1")
   )
   (sheet_instances
     (path "/" (page "1"))
   )
-  (symbol_instances
-    (path "/9fa81b1d-9622-4bc6-8198-4b4bc1b152f4"
-      (reference "J?") (unit 1) (value "Screw_Terminal_01x01") (footprint "")
-    )
-  )
 )
